Commit message: Add: object_frame in srdf, xrdf, urdf

File: dsr_cumotion/srdf/m1013_with_vgc10.srdf.xacro (robot description, xacro)
@@ -5,4 +5,8 @@
   <group name="manipulator">
     <chain base_link="base_link" tip_link="$(arg tcp_frame)"/>
+  </group>
+  <!-- Manipulator group definition -->
+  <group name="manipulator_object">
+    <chain base_link="base_link" tip_link="object_frame"/>
   </group>
   <!-- Predefined joint configurations -->
@@ -16,4 +20,20 @@
   </group_state>
   <group_state name="set" group="manipulator">
+    <joint name="joint_1" value="0"/>
+    <joint name="joint_2" value="0"/>
+    <joint name="joint_3" value="1.5708"/>
+    <joint name="joint_4" value="0"/>
+    <joint name="joint_5" value="1.5708"/>
+    <joint name="joint_6" value="0"/>
+  </group_state>
+  <group_state name="all-zeros" group="manipulator_object">
+    <joint name="joint_1" value="0"/>
+    <joint name="joint_2" value="0"/>
+    <joint name="joint_3" value="0"/>
+    <joint name="joint_4" value="0"/>
+    <joint name="joint_5" value="0"/>
+    <joint name="joint_6" value="0"/>
+  </group_state>
+  <group_state name="set" group="manipulator_object">
     <joint name="joint_1" value="0"/>
     <joint name="joint_2" value="0"/>
@@ -48,3 +68,4 @@
   <!-- Fixed: changed "Never" to "Adjacent" -->
   <disable_collisions link1="grasp_frame" link2="onrobot_vgc10_base_link" reason="Adjacent"/>
+  <disable_collisions link1="object_frame" link2="grasp_frame" reason="Adjacent"/>
 </robot>

File: dsr_cumotion/urdf/m1013_with_vgc10.urdf (robot description, URDF)
Before this commit: robot m1013, 17 links, 16 joints
Links:
- added link object_frame, mass 0.01
Joints:
- added joint object_joint: type fixed, parent grasp_frame, child object_frame, origin xyz=0 0 0.07 rpy=0 0 0

File: dsr_cumotion/urdf/m1013_with_vgc10.urdf.xacro (robot description, xacro)
@@ -36,4 +36,16 @@
     <child  link="grasp_frame"/>
   </joint>
+  <link name="object_frame">
+    <inertial>
+      <origin xyz="0 0 0" rpy="0 0 0"/>
+      <mass value="0.01"/>
+      <inertia ixx="0.0001" ixy="0.0" ixz="0.0" iyy="0.0001" iyz="0.0" izz="0.0001"/>
+    </inertial>
+  </link>
+  <joint name="object_joint" type="fixed">
+    <origin xyz="0 0 0.07" rpy="0 0 0"/>
+    <parent link="grasp_frame"/>
+    <child link="object_frame"/>
+  </joint>
   <!-- ros2_control -->
   <xacro:include filename="$(find dsr_cumotion)/urdf/m1013.ros2_control.xacro"/>
