Commit message: fix: obstacle handling, 2f85 SRDF call, and gripper joint orientation
- Fix obstacle manager function logic
- Fix missing robotiq 2F-85 SRDF macro invocation
- Fix robotiq 2F-85 gripper joint RPY orientation
- Apply serialized execution structure to prevent BaseExecutor stderr issues

File: dsr_cumotion/srdf/m1013.srdf.xacro (robot description, xacro)
@@ -52,4 +52,5 @@
   <xacro:if value="${gripper == '2f85'}">
     <xacro:include filename="$(find dsr_cumotion)/srdf/robotiq_2f_85.srdf.xacro"/>
+    <xacro:robotiq_2f85_srdf name="robotiq_2f85" prefix=""/>
     <disable_collisions link1="robotiq_85_base_link" link2="link_5" reason="Never"/>
     <disable_collisions link1="robotiq_85_base_link" link2="link_6" reason="Adjacent"/>

File: dsr_cumotion/urdf/robotiq/robotiq.xacro (robot description, xacro)
@@ -93,5 +93,5 @@
       <parent link="gripper_frame"/>
       <child  link="robotiq_85_base_link"/>
-      <origin xyz="0 0 0" rpy="0 0 0"/>
+      <origin xyz="0 0 0" rpy="0 0 1.57"/>
     </joint>
     <joint name="robotiq_85_left_knuckle_joint" type="revolute">
