Commit message: update: Refactor launch files for ROS 2 Jazzy and add JointTrajectoryController parameters
- Updated bringup and MoveIt-related launch files to follow Jazzy conventions
- Replaced deprecated launch actions and cleaned event sequencing
- Improved namespace handling and parameter injection
- Added full JointTrajectoryController configuration:
  - allow_nonzero_velocity_at_trajectory_end
  - interpolate_from_desired_state
  - allow_partial_joints_goal
  - constraints (goal_time, stopped_velocity_tolerance)

File: dsr_cumotion/urdf/m1013_with_vgc10.urdf.xacro (robot description, xacro)
@@ -48,4 +48,10 @@
     <child link="object_frame"/>
   </joint>
+  <link name="world"/>
+  <joint name="world_fixed" type="fixed">
+    <origin xyz="0 0 0" rpy="0 0 0"/>
+    <parent link="world"/>
+    <child  link="base_link"/>
+  </joint>
   <!-- ros2_control -->
   <xacro:include filename="$(find dsr_cumotion)/urdf/m1013.ros2_control.xacro"/>
