Commit message: - Added new ROS 2 Jazzy version of start_launch.py   (clean controller sequencing, namespace support, MoveIt2 integration) - Updated dsr_controller2.yaml with new parameters and Jazzy ros2_control format - Added cuMotion config files:   - object_attach.yaml   - param.yaml for cuMotion planner/action server - Updated RViz configuration (MoveIt2 panels, cuMotion visualizers, TF, tool frames) - Added Dockerfile and build-doosan.sh for automatic Isaac ROS + Doosan build - Added README.md with setup steps (docker/scripts, config.yaml, activate workflow)

File: dsr_cumotion/urdf/m1013.ros2_control.xacro (robot description, xacro)
@@ -1,67 +1,37 @@
 <?xml version="1.0"?>
 <robot xmlns:xacro="http://www.ros.org/wiki/xacro">
+  <!-- Doosan M1013 ros2_control (arm-only) -->
   <xacro:macro name="m1013_ros2_control" params="
-  name
-  host:=0.0.0.0
-  rt_host:=0.0.0.0
-  port:=12345
-  mode:=real
-  model:=m1013
-  ">
+      name
+      rate:=100
+      standby:=true
+      command:=none
+      host:=127.0.0.1
+      port:=12345
+      mode:=virtual
+      model:=m1013
+      mobile:=none">
+    <xacro:property name="double_pi" value="${2.0 * pi}"/>
+    <xacro:property name="neg_double_pi" value="${-2.0 * pi}"/>
     <ros2_control name="${name}" type="system">
       <hardware>
         <plugin>dsr_hardware2/DRHWInterface</plugin>
+        <!-- virtual 테스트면 true 유지 가능 (실기면 false 권장) -->
+        <param name="use_mock_hardware">false</param>
+        <param name="name">${name}</param>
+        <param name="rate">${rate}</param>
+        <param name="standby">${standby}</param>
+        <param name="command">${command}</param>
         <param name="host">${host}</param>
-        <param name="rt_host">${rt_host}</param>
         <param name="port">${port}</param>
         <param name="mode">${mode}</param>
         <param name="model">${model}</param>
+        <param name="mobile">${mobile}</param>
       </hardware>
+      <!-- Arm joints only -->
       <joint name="joint_1">
         <command_interface name="position">
-          <param name="min">{-2*pi}</param>
-          <param name="max">{2*pi}</param>
-        </command_interface>
-        <command_interface name="velocity">
-          <param name="min">-3.15</param>
-          <param name="max">3.15</param>
-        </command_interface>
-        <state_interface name="position">
-          <param name="initial_value">0.0</param>
-        </state_interface>
-        <state_interface name="velocity"/>
-      </joint>
-      <joint name="joint_2">
-        <command_interface name="position">
-          <param name="min">{-2*pi}</param>
-          <param name="max">{2*pi}</param>
-        </command_interface>
-        <command_interface name="velocity">
-          <param name="min">-3.15</param>
-          <param name="max">3.15</param>
-        </command_interface>
-        <state_interface name="position">
-          <param name="initial_value">0.0</param>
-        </state_interface>
-        <state_interface name="velocity"/>
-      </joint>
-      <joint name="joint_3">
-        <command_interface name="position">
-          <param name="min">{-pi}</param>
-          <param name="max">{pi}</param>
-        </command_interface>
-        <command_interface name="velocity">
-          <param name="min">-3.15</param>
-          <param name="max">3.15</param>
-        </command_interface>
-        <state_interface name="position">
-          <param name="initial_value">0.0</param>
-        </state_interface>
-        <state_interface name="velocity"/>
-      </joint>
-      <joint name="joint_4">
-        <command_interface name="position">
-          <param name="min">{-2*pi}</param>
-          <param name="max">{2*pi}</param>
+          <param name="min">${neg_double_pi}</param>
+          <param name="max">${double_pi}</param>
         </command_interface>
         <command_interface name="velocity">
@@ -69,13 +39,11 @@
           <param name="max">3.2</param>
         </command_interface>
-        <state_interface name="position">
-          <param name="initial_value">0.0</param>
-        </state_interface>
+        <state_interface name="position"><param name="initial_value">0.0</param></state_interface>
         <state_interface name="velocity"/>
       </joint>
-      <joint name="joint_5">
+      <joint name="joint_2">
         <command_interface name="position">
-          <param name="min">{-2*pi}</param>
-          <param name="max">{2*pi}</param>
+          <param name="min">${neg_double_pi}</param>
+          <param name="max">${double_pi}</param>
         </command_interface>
         <command_interface name="velocity">
@@ -83,13 +51,11 @@
           <param name="max">3.2</param>
         </command_interface>
-        <state_interface name="position">
-          <param name="initial_value">0.0</param>
-        </state_interface>
+        <state_interface name="position"><param name="initial_value">0.0</param></state_interface>
         <state_interface name="velocity"/>
       </joint>
-      <joint name="joint_6">
+      <joint name="joint_3">
         <command_interface name="position">
-          <param name="min">{-2*pi}</param>
-          <param name="max">{2*pi}</param>
+          <param name="min">${neg_double_pi}</param>
+          <param name="max">${double_pi}</param>
         </command_interface>
         <command_interface name="velocity">
@@ -97,7 +63,41 @@
           <param name="max">3.2</param>
         </command_interface>
-        <state_interface name="position">
-          <param name="initial_value">0.0</param>
-        </state_interface>
+        <state_interface name="position"><param name="initial_value">0.0</param></state_interface>
+        <state_interface name="velocity"/>
+      </joint>
+      <joint name="joint_4">
+        <command_interface name="position">
+          <param name="min">${neg_double_pi}</param>
+          <param name="max">${double_pi}</param>
+        </command_interface>
+        <command_interface name="velocity">
+          <param name="min">-3.2</param>
+          <param name="max">3.2</param>
+        </command_interface>
+        <state_interface name="position"><param name="initial_value">0.0</param></state_interface>
+        <state_interface name="velocity"/>
+      </joint>
+      <joint name="joint_5">
+        <command_interface name="position">
+          <param name="min">${neg_double_pi}</param>
+          <param name="max">${double_pi}</param>
+        </command_interface>
+        <command_interface name="velocity">
+          <param name="min">-3.2</param>
+          <param name="max">3.2</param>
+        </command_interface>
+        <state_interface name="position"><param name="initial_value">0.0</param></state_interface>
+        <state_interface name="velocity"/>
+      </joint>
+      <joint name="joint_6">
+        <command_interface name="position">
+          <param name="min">${neg_double_pi}</param>
+          <param name="max">${double_pi}</param>
+        </command_interface>
+        <command_interface name="velocity">
+          <param name="min">-3.2</param>
+          <param name="max">3.2</param>
+        </command_interface>
+        <state_interface name="position"><param name="initial_value">0.0</param></state_interface>
         <state_interface name="velocity"/>
       </joint>

File: dsr_cumotion/urdf/m1013_with_vgc10.urdf.xacro (robot description, xacro)
@@ -1,16 +1,17 @@
 <?xml version="1.0"?>
 <robot xmlns:xacro="http://www.ros.org/wiki/xacro" name="m1013_with_vgc10">
-  <xacro:arg name="color" default="white"/>
-  <xacro:arg name="namespace" default=""/>
+  <xacro:arg name="mode"           default="virtual"/>
+  <xacro:arg name="color"          default="white"/>
+  <xacro:arg name="namespace"      default=""/>
+  <!-- gripper control argument -->
+  <xacro:arg name="gripper"              default="none"/>
   <xacro:arg name="use_gazebo" default="false"/>
-  <xacro:arg name="host" default=""/>
-  <xacro:arg name="port" default=""/>
-  <xacro:arg name="rt_host" default=""/>
-  <xacro:arg name="mode" default=""/>
-  <xacro:arg name="model" default="m1013"/>
+  <xacro:property name="gz" value="$(arg use_gazebo)"/>
+  <xacro:property name="cr" value="$(arg color)"/>
+  <xacro:property name="gr" value="$(arg gripper)"/>
   <xacro:include filename="$(find dsr_cumotion)/urdf/macro.m1013.white.xacro"/>
   <xacro:m1013 namespace="$(arg namespace)"/>
   <link name="tool0"/>
-  <joint name="joint_6-tool0" type="fixed">
+  <joint name="joint6-tool0" type="fixed">
     <origin xyz="0 0 0" rpy="0 0 0"/>
     <parent link="link_6"/>
@@ -25,4 +26,10 @@
   </joint>
   <xacro:include filename="$(find dsr_cumotion)/urdf/vgc10/onrobot_vgc10_4cups_model.urdf"/>
+  <link name="world"/>
+  <joint name="world_fixed" type="fixed">
+    <origin xyz="0 0 0" rpy="0 0 0"/>
+    <parent link="world"/>
+    <child  link="base_link"/>
+  </joint>
   <joint name="gripper_to_vgc10" type="fixed">
     <origin xyz="0 0 0" rpy="0 0 0"/>
@@ -48,18 +55,6 @@
     <child link="object_frame"/>
   </joint>
-  <link name="world"/>
-  <joint name="world_fixed" type="fixed">
-    <origin xyz="0 0 0" rpy="0 0 0"/>
-    <parent link="world"/>
-    <child  link="base_link"/>
-  </joint>
   <!-- ros2_control -->
   <xacro:include filename="$(find dsr_cumotion)/urdf/m1013.ros2_control.xacro"/>
-  <xacro:m1013_ros2_control
-    name="m1013"
-    host="$(arg host)"
-    rt_host="$(arg rt_host)"
-    port="$(arg port)"
-    mode="$(arg mode)"
-    model="$(arg model)"/>
+  <xacro:m1013_ros2_control name="m1013"/>
 </robot>

File: dsr_cumotion/urdf/macro.m1013.white.xacro (robot description, xacro)
@@ -2,6 +2,6 @@
 <robot name="m1013" xmlns:xacro="http://www.ros.org/wiki/xacro">
   <!-- dependencies -->
-  <xacro:include filename="$(find dsr_description2)/config/macro.gazebo.xacro"/>
-  <xacro:include filename="$(find dsr_description2)/config/macro.transmission.xacro"/>
+  <!-- <xacro:include filename="$(find dsr_description2)/config/macro.gazebo.xacro"/>
+  <xacro:include filename="$(find dsr_description2)/config/macro.transmission.xacro"/> -->
   <xacro:include filename="$(find dsr_description2)/config/macro.materials.xacro"/>
   <xacro:property name="vision_bracket_mesh"
@@ -262,6 +262,6 @@
       </visual>
     </link> -->
-    <xacro:dsr_transmission/>
-    <xacro:dsr_gazebo namespace="${namespace}"/>
+    <!-- <xacro:dsr_transmission/> -->
+    <!-- <xacro:dsr_gazebo namespace="${namespace}"/> -->
   </xacro:macro>
 </robot>
