Commit message: hotfix: Fix link6 and tool0 tf matching

File: dsr_cumotion/urdf/m1013_with_vgc10.urdf (robot description, URDF)
Before this commit: robot m1013, 18 links, 17 joints
Joints:
- joint joint_6-tool0: origin xyz=0 0 0 rpy=0 0 1.57 -> xyz=0 0 0 rpy=0 0 0

File: dsr_cumotion/urdf/m1013_with_vgc10.urdf.xacro (robot description, xacro)
@@ -13,5 +13,5 @@
   <link name="tool0"/>
   <joint name="joint_6-tool0" type="fixed">
-    <origin xyz="0 0 0" rpy="0 0 1.57"/>
+    <origin xyz="0 0 0" rpy="0 0 0"/>
     <parent link="link_6"/>
     <child link="tool0"/>

Commit message: ADD: urdf args

File: dsr_cumotion/urdf/m1013_with_vgc10.urdf (robot description, URDF)
Before this commit: robot m1013, 17 links, 16 joints
Links:
- removed link base
- added link object_frame, mass 0.01
- link base_link: mass 3.722 -> 4.12; geometry collision mesh filename=package://dsr_cumotion/meshes/m1013_collision/MF1013_0_0.dae scale=0.001 0.001 0.001; visual mesh filename=package://dsr_cumotion/meshes/m1013_white/MF1013_0_0.dae scale=0.001 0.001 0.001
- link gripper_frame: mass 0.01 -> None
- link link_1: mass 7.446 -> 7.8; geometry collision mesh filename=package://dsr_cumotion/meshes/m1013_collision/MF1013_1_0.dae scale=0.001 0.001 0.001; visual mesh filename=package://dsr_cumotion/meshes/m1013_white/MF1013_1_0.dae scale=0.001 0.001 0.001
- link link_2: mass 10.569 -> 10.83; geometry collision mesh filename=package://dsr_cumotion/meshes/m1013_collision/MF1013_2_0.dae scale=0.001 0.001 0.001; collision mesh filename=package://dsr_cumotion/meshes/m1013_collision/MF1013_2_1.dae scale=0.001 0.001 0.001
- link link_3: mass 3.614 -> 3.68; geometry collision mesh filename=package://dsr_cumotion/meshes/m1013_collision/MF1013_3_0.dae scale=0.001 0.001 0.001; visual mesh filename=package://dsr_cumotion/meshes/m1013_white/MF1013_3_0.dae scale=0.001 0.001 0.001
- link link_4: mass 3.785 -> 3.82; geometry collision mesh filename=package://dsr_cumotion/meshes/m1013_collision/MF1013_4_0.dae scale=0.001 0.001 0.001; collision mesh filename=package://dsr_cumotion/meshes/m1013_collision/MF1013_4_1.dae scale=0.001 0.001 0.001
- link link_5: mass 2.598 -> 2.82; geometry collision mesh filename=package://dsr_cumotion/meshes/m1013_collision/MF1013_5_0.dae scale=0.001 0.001 0.001; visual mesh filename=package://dsr_cumotion/meshes/m1013_white/MF1013_5_0.dae scale=0.001 0.001 0.001
- link link_6: mass 1.128 -> 1.16; geometry collision mesh filename=package://dsr_cumotion/meshes/m1013_collision/MF1013_6_0.dae scale=0.001 0.001 0.001; visual mesh filename=package://dsr_cumotion/meshes/m1013_white/MF1013_6_0.dae scale=0.001 0.001 0.001
- link suction1: mass None -> 0.2
- link suction2: mass None -> 0.2
- link suction3: mass None -> 0.2
- link suction4: mass None -> 0.2
Joints:
- removed joint base_link-base
- removed joint gripper_joint
- added joint object_joint: type fixed, parent grasp_frame, child object_frame, origin xyz=0 0 0.07 rpy=0 0 0
- added joint tool0_to_gripper_frame: type fixed, parent tool0, child gripper_frame, origin xyz=0 0 0 rpy=0 0 0
- joint _suction1_joint: axis (none) -> 1 0 0; origin xyz=0.0175 0.0175 0 rpy=0 0 0 -> xyz=0.0175 0.0175 0. rpy=0 0 0
- joint _suction2_joint: axis (none) -> 1 0 0; origin xyz=0.0175 -0.0175 0 rpy=0 0 0 -> xyz=0.0175 -0.0175 0. rpy=0 0 0
- joint _suction3_joint: axis (none) -> 1 0 0; origin xyz=-0.0175 0.0175 0 rpy=0 0 0 -> xyz=-0.0175 0.0175 0. rpy=0 0 0
- joint _suction4_joint: axis (none) -> 1 0 0; origin xyz=-0.0175 -0.0175 0 rpy=0 0 0 -> xyz=-0.0175 -0.0175 0. rpy=0 0 0
- joint _suction_joint: axis (none) -> 1 0 0; origin xyz=0 0 0.0835 rpy=0 0 0 -> xyz=0. 0. 0.08350 rpy=0 0 0
- joint joint_1: limit lower=-2.1 upper=2.1 effort=20400 velocity=1.571 -> lower=-1.3 upper=2.0 effort=346 velocity=2.0944
- joint joint_2: limit lower=-4.0 upper=1.0 effort=20400 velocity=1.571 -> lower=-6.2832 upper=6.2832 effort=346 velocity=2.0944
- joint joint_3: limit lower=-2.4 upper=2.4 effort=9600 velocity=1.571 -> lower=-0.01 upper=2.7925 effort=163 velocity=3.1416
- joint joint_4: limit lower=-6.283 upper=6.283 effort=2700 velocity=1.571 -> lower=-3.14 upper=3.14 effort=50 velocity=3.927
- joint joint_5: limit lower=-2.356 upper=2.356 effort=2700 velocity=1.571 -> lower=-2.0 upper=2.0 effort=50 velocity=3.927
- joint joint_6: limit lower=-6.283 upper=6.283 effort=2700 velocity=1.571 -> lower=-3.14 upper=3.14 effort=50 velocity=3.927
- joint joint_6-tool0: origin xyz=0 0 0 rpy=0 0 1.57 -> xyz=0 0 0 rpy=0 0 0

File: dsr_cumotion/urdf/m1013_with_vgc10.urdf.xacro (robot description, xacro)
@@ -1,17 +1,20 @@
 <?xml version="1.0"?>
 <robot xmlns:xacro="http://www.ros.org/wiki/xacro" name="m1013_with_vgc10">
-  <xacro:arg name="color" default="white"/>
-  <xacro:arg name="namespace" default=""/>
-  <xacro:arg name="use_gazebo" default="false"/>
-  <xacro:arg name="host" default=""/>
-  <xacro:arg name="port" default=""/>
-  <xacro:arg name="rt_host" default=""/>
-  <xacro:arg name="mode" default=""/>
-  <xacro:arg name="model" default="m1013"/>
+  <xacro:arg name="color"        default="white"/>
+  <xacro:arg name="gripper"      default="none"/>
+  <xacro:arg name="namespace"    default=""/>
+  <xacro:arg name="use_gazebo"   default="false"/>
+  <xacro:arg name="use_mujoco"   default="false"/>
+  <xacro:arg name="host"         default=""/>
+  <xacro:arg name="port"         default=""/>
+  <xacro:arg name="rt_host"      default=""/>
+  <xacro:arg name="mode"         default=""/>
+  <xacro:arg name="model"        default=""/>
+  <xacro:arg name="update_rate"  default=""/>
   <xacro:include filename="$(find dsr_cumotion)/urdf/macro.m1013.white.xacro"/>
   <xacro:m1013 namespace="$(arg namespace)"/>
   <link name="tool0"/>
   <joint name="joint_6-tool0" type="fixed">
-    <origin xyz="0 0 0" rpy="0 0 1.57"/>
+    <origin xyz="0 0 0" rpy="0 0 0"/>
     <parent link="link_6"/>
     <child link="tool0"/>
@@ -36,4 +39,16 @@
     <child  link="grasp_frame"/>
   </joint>
+  <link name="object_frame">
+    <inertial>
+      <origin xyz="0 0 0" rpy="0 0 0"/>
+      <mass value="0.01"/>
+      <inertia ixx="0.0001" ixy="0.0" ixz="0.0" iyy="0.0001" iyz="0.0" izz="0.0001"/>
+    </inertial>
+  </link>
+  <joint name="object_joint" type="fixed">
+    <origin xyz="0 0 0.07" rpy="0 0 0"/>
+    <parent link="grasp_frame"/>
+    <child link="object_frame"/>
+  </joint>
   <!-- ros2_control -->
   <xacro:include filename="$(find dsr_cumotion)/urdf/m1013.ros2_control.xacro"/>
@@ -44,4 +59,5 @@
     port="$(arg port)"
     mode="$(arg mode)"
-    model="$(arg model)"/>
+    model="$(arg model)"
+    update_rate="$(arg update_rate)"/>
 </robot>

File: dsr_cumotion/urdf/m1013_without_gripper.urdf (robot description, URDF)
Before this commit: robot m1013, 11 links, 10 joints
Links:
- removed link base
- added link world
- link base_link: mass 3.722 -> 4.12; geometry collision mesh filename=package://dsr_cumotion/meshes/m1013_collision/MF1013_0_0.dae scale=0.001 0.001 0.001; visual mesh filename=package://dsr_cumotion/meshes/m1013_white/MF1013_0_0.dae scale=0.001 0.001 0.001
- link link_1: mass 7.446 -> 7.8; geometry collision mesh filename=package://dsr_cumotion/meshes/m1013_collision/MF1013_1_0.dae scale=0.001 0.001 0.001; visual mesh filename=package://dsr_cumotion/meshes/m1013_white/MF1013_1_0.dae scale=0.001 0.001 0.001
- link link_2: mass 10.569 -> 10.83; geometry collision mesh filename=package://dsr_cumotion/meshes/m1013_collision/MF1013_2_0.dae scale=0.001 0.001 0.001; collision mesh filename=package://dsr_cumotion/meshes/m1013_collision/MF1013_2_1.dae scale=0.001 0.001 0.001
- link link_3: mass 3.614 -> 3.68; geometry collision mesh filename=package://dsr_cumotion/meshes/m1013_collision/MF1013_3_0.dae scale=0.001 0.001 0.001; visual mesh filename=package://dsr_cumotion/meshes/m1013_white/MF1013_3_0.dae scale=0.001 0.001 0.001
- link link_4: mass 3.785 -> 3.82; geometry collision mesh filename=package://dsr_cumotion/meshes/m1013_collision/MF1013_4_0.dae scale=0.001 0.001 0.001; collision mesh filename=package://dsr_cumotion/meshes/m1013_collision/MF1013_4_1.dae scale=0.001 0.001 0.001
- link link_5: mass 2.598 -> 2.82; geometry collision mesh filename=package://dsr_cumotion/meshes/m1013_collision/MF1013_5_0.dae scale=0.001 0.001 0.001; visual mesh filename=package://dsr_cumotion/meshes/m1013_white/MF1013_5_0.dae scale=0.001 0.001 0.001
- link link_6: mass 1.128 -> 1.16; geometry collision mesh filename=package://dsr_cumotion/meshes/m1013_collision/MF1013_6_0.dae scale=0.001 0.001 0.001; visual mesh filename=package://dsr_cumotion/meshes/m1013_white/MF1013_6_0.dae scale=0.001 0.001 0.001
Joints:
- removed joint base_link-base
- added joint world_fixed: type fixed, parent world, child base_link, origin xyz=0 0 0 rpy=0 0 0
- joint joint_1: limit lower=-2.1 upper=2.1 effort=20400 velocity=1.571 -> lower=-6.2832 upper=6.2832 effort=346 velocity=2.0944
- joint joint_2: limit lower=-4.0 upper=1.0 effort=20400 velocity=1.571 -> lower=-6.2832 upper=6.2832 effort=346 velocity=2.0944
- joint joint_3: limit lower=-2.4 upper=2.4 effort=9600 velocity=1.571 -> lower=-0.1 upper=2.7925 effort=163 velocity=3.1416
- joint joint_4: limit lower=-6.283 upper=6.283 effort=2700 velocity=1.571 -> lower=-6.2832 upper=6.2832 effort=50 velocity=3.927
- joint joint_5: limit lower=-2.356 upper=2.356 effort=2700 velocity=1.571 -> lower=-6.2832 upper=6.2832 effort=50 velocity=3.927
- joint joint_6: limit lower=-6.283 upper=6.283 effort=2700 velocity=1.571 -> lower=-6.2832 upper=6.2832 effort=50 velocity=3.927

File: dsr_cumotion/urdf/m1013_without_gripper.urdf.xacro (robot description, xacro)
@@ -14,5 +14,4 @@
   <xacro:arg name="gripper_prefix"      default=""/>
   <xacro:arg name="gripper_parent_link" default="vision_bracket"/>
-   world → base_link
   <link name="world"/>
   <joint name="world_fixed" type="fixed">
