Commit message: feat: Add gripper support for 2f85 and vgc10 models with mode restriction
- Added support for 2f85 and vgc10 gripper models
- Updated URDF, SRDF, and XACRO files with new gripper arguments
- Restricted 2F85 gripper usage to VIRTUAL mode only due to controller limitations
- Added validation function to block invalid mode/gripper combinations

File: dsr_cumotion/urdf/m1013_with_2f85.urdf (robot description, URDF)
Before this commit: robot m1013, 22 links, 21 joints
Links:
- removed link d435i_camera
- removed link vision_bracket
Joints:
- removed joint d435i_camera_joint
- removed joint vision_bracket_joint
- joint gripper_joint: parent robotiq_85_base_link -> tool0
- joint robotiq_85_base_joint: parent vision_bracket -> gripper_frame

File: dsr_cumotion/urdf/m1013_with_vgc10.urdf (robot description, URDF)
Before this commit: robot m1013_with_vgc10, 17 links, 16 joints
Joints:
- removed joint tool0_to_gripper_frame
- added joint gripper_joint: type fixed, parent tool0, child gripper_frame, origin xyz=0 0 0 rpy=0 0 0

File: dsr_cumotion/urdf/macro.m1013.white.xacro (robot description, xacro)
@@ -236,4 +236,17 @@
       </visual>
     </link>
+    <link name="tool0"/>
+    <joint name="joint_6-tool0" type="fixed">
+      <origin xyz="0 0 0" rpy="0 0 0"/>
+      <parent link="link_6"/>
+      <child link="tool0"/>
+    </joint>
+    <!-- Gripper Frame -->
+    <link name="gripper_frame"/>
+    <joint name="gripper_joint" type="fixed">
+      <origin xyz="0 0 0" rpy="0 0 0"/>
+      <parent link="tool0"/>
+      <child  link="gripper_frame"/>
+    </joint>
     <!-- <joint name="vision_bracket_joint" type="fixed">
       <parent link="tool0"/>

File: dsr_cumotion/urdf/robotiq/robotiq.xacro (robot description, xacro)
@@ -1,5 +1,5 @@
 <?xml version="1.0"?>
 <robot xmlns:xacro="http://www.ros.org/wiki/xacro">
-  <xacro:macro name="robotiq_85" params="parent prefix base_xyz:='0 0 0' base_rpy:='0 0 0'">
+  <xacro:macro name="robotiq_85">
     <!-- base -->
     <link name="robotiq_85_base_link">
@@ -23,5 +23,5 @@
     </link>
     <link name="robotiq_85_right_knuckle_link">
-      <visual><geometry><mesh filename="package://dsr_cumotion//meshes/gripper/robotiq/2f85/visual/right_knuckle.dae"/></geometry></visual>
+      <visual><geometry><mesh filename="package://dsr_cumotion/meshes/gripper/robotiq/2f85/visual/right_knuckle.dae"/></geometry></visual>
       <collision><geometry><mesh filename="package://dsr_cumotion/meshes/gripper/robotiq/2f85/collision/right_knuckle.stl"/></geometry></collision>
       <inertial>
@@ -90,7 +90,6 @@
       </inertial>
     </link>
-    <!-- joints: gripper base fixed to vision_bracket -->
     <joint name="robotiq_85_base_joint" type="fixed">
-      <parent link="vision_bracket"/>
+      <parent link="gripper_frame"/>
       <child  link="robotiq_85_base_link"/>
       <origin xyz="0 0 0" rpy="0 0 0"/>
@@ -153,16 +152,4 @@
       <mimic joint="robotiq_85_left_knuckle_joint" multiplier="1" offset="0.0"/>
     </joint>
-    <link name="gripper_frame">
-      <inertial>
-        <origin xyz="0 0 0" rpy="0 0 0"/>
-        <mass value="0.01"/>
-        <inertia ixx="0.0001" ixy="0.0" ixz="0.0" iyy="0.0001" iyz="0.0" izz="0.0001"/>
-      </inertial>
-    </link>
-    <joint name="gripper_joint" type="fixed">
-      <origin rpy="0 0 0" xyz="0 0 0"/>
-      <parent link="robotiq_85_base_link"/>
-      <child  link="gripper_frame"/>
-    </joint>
     <link name="grasp_frame">
       <inertial>

File: dsr_cumotion/urdf/vgc10/onrobot_vgc10_4cups_model.urdf (robot description, URDF)
Before this commit: robot onrobot_vgc10_model, 6 links, 5 joints
Links:
- added link grasp_frame
- added link object_frame, mass 0.01
Joints:
- added joint grasp_joint: type fixed, parent gripper_frame, child grasp_frame, origin xyz=0 0 0.12 rpy=0 0 0
- added joint gripper_to_vgc10: type fixed, parent gripper_frame, child onrobot_vgc10_base_link, origin xyz=0 0 0 rpy=0 0 0
- added joint object_joint: type fixed, parent grasp_frame, child object_frame, origin xyz=0 0 0.07 rpy=0 0 0
